Commit message: Debugging

File: qube_description/urdf/qube.macro.xacro (robot description, xacro)
@@ -2,5 +2,4 @@
 <robot xmlns:xacro="http://www.ros.org/wiki/xacro">
   <xacro:macro name="qube" params="prefix">
-    <!-- Dimensjoner -->
     <xacro:property name="base_size" value="0.102"/>
     <xacro:property name="disk_radius" value="0.025"/>
@@ -9,7 +8,5 @@
     <xacro:property name="indicator_width" value="0.002"/>
     <xacro:property name="indicator_height" value="0.002"/>
-    <!-- base_link -->
     <link name="${prefix}base_link"/>
-    <!-- svart boks -->
     <link name="${prefix}stator_link">
       <visual>
@@ -23,8 +20,7 @@
       </visual>
     </link>
-    <!-- rød disk -->
     <link name="${prefix}rotor_link">
       <visual>
-        <origin xyz="0 0 0" rpy="1.5708 0 0"/>
+        <origin xyz="0 0 0" rpy="0 0 0"/>
         <geometry>
           <cylinder radius="${disk_radius}" length="${disk_height}"/>
@@ -35,5 +31,4 @@
       </visual>
     </link>
-    <!-- hvit viser -->
     <link name="${prefix}angle_link">
       <visual>
@@ -47,5 +42,4 @@
       </visual>
     </link>
-    <!-- base_link -> stator -->
     <joint name="${prefix}stator_joint" type="fixed">
       <parent link="${prefix}base_link"/>
@@ -53,12 +47,10 @@
       <origin xyz="0 0 0" rpy="0 0 0"/>
     </joint>
-    <!-- stator -> rotor -->
     <joint name="${prefix}motor_joint" type="continuous">
       <parent link="${prefix}stator_link"/>
       <child link="${prefix}rotor_link"/>
       <origin xyz="0 0 ${base_size}" rpy="0 0 0"/>
-      <axis xyz="0 0 1"/>
+      <axis xyz="0 0 -1"/>
     </joint>
-    <!-- rotor -> angle -->
     <joint name="${prefix}indicator_joint" type="fixed">
       <parent link="${prefix}rotor_link"/>
